File: Hardware/ButterflyBadge/PortWing.kicad_sch (KiCad schematic)
At the start: 266 parts, among them J1 Conn_01x06, J4 Conn_01x08, U1 XC6206PxxxMR, U5 SN74LV1T34DBV

Commit message: Schematic is done! Now to work on the main PCB
Parts:
- removed ? (x3): (no value), symbol Device:C
- removed J1: Conn_01x06, symbol Connector_Generic:Conn_01x06
- added C35 (x3): C, symbol Device:C
- added X1: Badgelife_sao_connector_v169bis, badgelife_sao_v169bis:Badgelife-SAOv169-BADGE-2x3, symbol badgelife_shitty_addon_v169bis:Badgelife_sao_connector_v169bis
- ?: now fitted
Connections:
- net 3V3: now also C35.1, C35.1, X1.1 (VCC)
- net 5V: now also C35.1
- net GND: now also C35.2, C35.2, C35.2, X1.2 (GND)
- net NFC_MSG: now also X1.6 (GPIO2)
- net PORT_GP0: now also X1.5 (GPIO1)
- net SCL: now also X1.4 (SCL)
- net SDA: now also X1.3 (SDA)

Commit message: Hardware mods
Parts:
- ?: Manufacturer PN ST25DV04K-IER6S3 -> (none)
- D2: Manufacturer PN C2890364 -> (none)
