File: Hardware/ButterflyBadge/ButterflyBadge.kicad_sch (KiCad schematic)
At the start: 9 parts

Commit message: Finished the power section
Parts:
- added C? (x4): C, symbol Device:C
- added C?: 22u, symbol Device:C
- added C?: 10u, symbol Device:C
- added D? (x2): D_Schottky, symbol Device:D_Schottky
- added D?: LED, symbol Device:LED
- added L?: L_Small, symbol Device:L_Small
- added R? (x2): R, symbol Device:R
- added R?: 7.68K, symbol Device:R
- added R? (x2): 5.1k, symbol Device:R
- added R?: 1K, symbol Device:R
- added SW?: SW_SPST, symbol Switch:SW_SPST
- added U?: AMS1117-3.3, Package_TO_SOT_SMD:SOT-223-3_TabPin2, symbol Regulator_Linear:AMS1117-3.3
- added U?: CN3058, symbol CN3058:CN3058
- added U?: MT3608, Package_TO_SOT_SMD:SOT-23-6, symbol Regulator_Switching:MT3608
- added U?: TMI8118, Package_TO_SOT_SMD:SOT-23-6, symbol TMI8118:TMI8118
Connections:
- net GND: now reaches J?.A1 (GND), J?.A12 (GND), J?.B1 (GND), J?.B12 (GND)
- net GND: now also BT?.2 (-), J?.S1 (SHIELD), C?.2, C?.2, C?.2, C?.2, C?.2, C?.2, R?.2, R?.2, R?.2, R?.2, U?.1 (GND), U?.1 (TEMP), U?.2 (GND), U?.3 (GND)
- net at J?.A4 (VBUS), J?.A9 (VBUS), J?.B4 (VBUS)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: now also D?.2 (A), U?.4 (VIN)
- net at J?.A5 (CC1): now also R?.1
- net USB_D+: now reaches J?.A6 (D+)
- net USB_D+: now also J?.B6 (D+)
- net USB_D-: now reaches J?.A7 (D-)
- net USB_D-: now also J?.B7 (D-)
- net at J?.B5 (CC2): now also R?.1
- net at BT?.1 (+): now also C?.1, C?.1, L?.1, U?.5 (BAT), U?.5 (IN), U?.8 (FB)
- new net: D?.2 (A), L?.2, U?.1 (SW)
- new net: R?.1, R?.2, U?.4 (EN)
- new net: C?.1, C?.1, D?.1 (K), D?.1 (K), R?.1, SW?.1 (A)
- new net: R?.1, R?.2, U?.3 (FB)
- new net: C?.1, U?.2 (VO)
- new net +5V: C?.1, R?.1, SW?.2 (B), U?.3 (VI)
Other:
- note added: "Vout = Vref (0.6V) * (1+(R1/R2(gndSide)) 5.2 = 0.6*(1+ (R/1K)) R1=7.6K=7.68K"
- moved on the sheet: BT?, J?

Commit message: More hardware work
Parts:
- removed U?: MT3608, Package_TO_SOT_SMD:SOT-23-6, symbol Regulator_Switching:MT3608
- added AE?: Antenna_Loop, symbol Device:Antenna_Loop
- added C? (x14): C, symbol Device:C
- added C?: 22u, symbol Device:C
- added R? (x3): R, symbol Device:R
- added SW?: SW_Push, symbol Switch:SW_Push
- added U?: W25Q128JVS, Package_SO:SOIC-8_5.23x5.23mm_P1.27mm, symbol Memory_Flash:W25Q128JVS
- added U?: AX5201, symbol Ax5201:AX5201
- added Y?: Crystal, symbol Device:Crystal
- R?: value 7.68K -> 4.22K
Connections:
- net +5V: now also U?.5 (VDD), C?.1
- net GND: now also P?.5 (GND), U?.19 (TESTEN), U?.2 (GND), U?.3 (GND), U?.4 (VSS), U?.57 (GND), C?.1, C?.2, C?.2, C?.2, C?.2, C?.2, C?.2, C?.2, C?.2, C?.2, C?.2, C?.2, C?.2, C?.2, R?.2, SW?.1, U?.4 (GND), U?.7 (PGND), U?.8 (SGND)
- net USB_D+: now also U?.46 (USB_DM)
- net USB_D-: now also U?.47 (USB_DP)
- net at BT?.1 (+), C?.1, C?.1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: now also U?.2 (VCC)
- net at D?.2 (A), L?.2: now also U?.5 (SW), U?.6 (SW), U?.9 (SW)
- net +3V3: now reaches U?.1 (VCC)
- net +3V3: now also C?.1, P?.1 (VCC), Q?.1 (C), U?.1 (IOVDD), U?.10 (IOVDD), U?.2 (VO), U?.22 (IOVDD), U?.33 (IOVDD), U?.42 (IOVDD), U?.43 (ADC_AVDD), U?.44 (VREG_IN), U?.48 (USB_VDD), U?.49 (IOVDD), U?.8 (VCC), C?.1, C?.1, C?.1, C?.1, C?.1, R?.2, U?.8 (VCC)
- net HALL_SENSOR: now reaches U?.2 (OUTPUT)
- net at R?.1, R?.2: now also U?.1 (EN)
- net at M?.1 (+): now also U?.1 (OUTB), C?.1, C?.2
- net at M?.2 (-): now also U?.6 (OUTA), C?.1, C?.2
- net at R?.1, R?.2: now also U?.3 (FB)
- net at U?.20 (XIN): now also C?.1, Y?.2
- net at U?.21 (XOUT): now also C?.1, Y?.1
- net at U?.24 (SWCLK): now also P?.4 (SWCLK/TCK)
- net at U?.25 (SWD): now also P?.2 (SWDIO/TMS)
- net RST: now reaches U?.26 (RUN)
- net RST: now also P?.3 (~{RESET}), R?.1
- net +1V1: now reaches U?.45 (VREG_VOUT)
- net +1V1: now also C?.1, C?.1, C?.1
- net at U?.51 (QSPI_SD3): now also U?.7 (IO3)
- net at U?.52 (QSPI_SCLK): now also U?.6 (CLK)
- net at U?.53 (QSPI_SD0): now also U?.5 (DI(IO0))
- net at U?.54 (QSPI_SD2): now also U?.3 (IO2)
- net at U?.55 (QSPI_SD1): now also U?.2 (DO(IO1))
- net at U?.56 (QSPI_SS): now also R?.2, U?.1 (~{CS})
- net at U?.2 (AC0): now also AE?.1
- net at U?.3 (AC1): now also AE?.2
- net SDA: now reaches U?.5 (SDA)
- net SCL: now reaches U?.6 (SCL)
- net NFC_MSG: now reaches U?.7 (GP0)
- net MOTOR_A: now reaches U?.3 (INB)
- net MOTOR_B: now reaches U?.4 (INA)
- net AMBIENT_LIGHT: now reaches Q?.2 (E)
- net AMBIENT_LIGHT: now also R?.1
- new net: R?.1, SW?.2
- new net: C?.1, U?.4 (SS)
Other:
- note added: "Saturation V 0.4V Saturation output voltage 4.6 need to detect between 35,000 and 18 lux 4K7 looks right"
- note added: "Vout = Vref (1) * (1+(R1/R2(gndSide)) R2= 1K~3K 5.2 = 1*(1+ (R/1K)) R1=4.22K"
- note removed: "Vout = Vref (0.6V) * (1+(R1/R2(gndSide)) 5.2 = 0.6*(1+ (R/1K)) R1=7.6K=7.68K"
- moved on the sheet: C?, D?, L?, M?, P?, R?, SW?, U?

Commit message: More schetaic work
Parts:
- removed AE?: Antenna_Loop, symbol Device:Antenna_Loop
- removed C?: C, symbol Device:C
- removed U?: ST25DV04K, Package_SO:SOIC-8-1EP_3.9x4.9mm_P1.27mm_EP2.41x3.3mm, symbol ST25DV04K:ST25DV04K
- added AE1: Antenna, symbol Device:Antenna
- added C1, C2 (x2), C4 (x4), C8 (x2): C, symbol Device:C
- added J1: Conn_01x10_Female, symbol Connector:Conn_01x10_Female
- added L1 (x3): L_Small, symbol Device:L_Small
- added R1, R2: R, symbol Device:R
- added U1: QSE159, OptoDevice:ONSemi_QSE15x, symbol Interface_Optical:QSE159
- added Y1: Crystal, symbol Device:Crystal
- ? (x13): renamed from C?; value C -> (none)
- ?: renamed from L?; value L_Small -> (none)
- ?: renamed from U?; value SM351LT -> (none); footprint Package_TO_SOT_SMD:SOT-23 -> (none)
- ?: renamed from J?; value USB_C_Receptacle_USB2.0 -> (none)
- ? (x5): renamed from R?; value R -> (none)
- ? (x4): renamed from C?; value C -> (none); now not fitted
- ?: renamed from M?; value Motor_DC -> (none)
- ?: renamed from U?; value W25Q128JVS -> (none); footprint Package_SO:SOIC-8_5.23x5.23mm_P1.27mm -> (none); now not fitted
- ?: renamed from R?; value 4.22K -> (none)
- ?: renamed from U?; value AMS1117-3.3 -> (none); footprint Package_TO_SOT_SMD:SOT-223-3_TabPin2 -> (none); now not fitted
- ?: renamed from U?; value RP2040 -> (none); footprint Package_DFN_QFN:QFN-56-1EP_7x7mm_P0.4mm_EP3.2x3.2mm -> (none)
- ?: renamed from U?; value Si24R1 -> (none); footprint Package_DFN_QFN:QFN-20-1EP_4x4mm_P0.5mm_EP2.5x2.5mm -> (none)
- ?: renamed from R?; value 5.1k -> (none)
- ? (x2): renamed from C?; value 22u -> (none)
- ?: renamed from C?; value 10u -> (none); now not fitted
- ?: renamed from SW?; value SW_Push -> (none)
- ? (x2): renamed from D?; value D_Schottky -> (none)
- ?: renamed from R?; value 5.1k -> (none); now not fitted
- ?: renamed from D?; value LED -> (none)
- ?: renamed from P?; value TC2030-CTX -> (none)
- ?: renamed from U?; value AX5201 -> (none)
- ?: renamed from SW?; value SW_SPST -> (none); now not fitted
- ?: renamed from BT?; value Battery_Cell -> (none)
- ?: renamed from U?; value CN3058 -> (none); now not fitted
- ?: renamed from Y?; value Crystal -> (none)
- ?: renamed from U?; value TMI8118 -> (none); footprint Package_TO_SOT_SMD:SOT-23-6 -> (none)
- ?: renamed from Q?; value ALS-PT19 -> (none); footprint ButterflyBadge:ALS-PT19-315C -> (none)
- ?: renamed from R?; value 1K -> (none)
Connections:
- net +3V3: now also ?.15 (VDD), ?.18 (VDD), ?.7 (VDD), C8.1, C8.1
- net +5V: now also J1.1 (Pin_1), J1.2 (Pin_2)
- net GND: now also ?.14 (VSS), ?.17 (VSS), ?.20 (VSS), ?.8 (VSS), C1.2, C2.2, C2.2, C4.1, C4.1, C4.1, C8.2, C8.2, J1.10 (Pin_10), J1.9 (Pin_9), R1.2
- net NRF_CE: now reaches ?.1 (CE)
- net at ?.10 (XC1): now also R2.1, Y1.2
- net at ?.11 (VDD_PA): now also C4.2, C4.2, L1.1
- net at ?.12 (ANT1): now also L1.1, L1.2
- net at ?.13 (ANT2): now also L1.1, L1.2
- net at ?.16 (IREF): now also R1.1
- net at ?.19 (DVDD): now also C1.1
- net NRF_CS: now reaches ?.2 (CSN)
- net SCK: now reaches ?.3 (SCK)
- net COPI: now reaches ?.4 (MOSI)
- net CIPO: now reaches ?.5 (MISO)
- net NRF_IRQ: now reaches ?.6 (IRQ)
- net at ?.9 (XC2): now also C2.1, C2.1, R2.2, Y1.1
- new net: AE1.1 (A), C4.2, C4.2
- new net: C4.1, L1.2
Other:
- added sheet LeftWing (LeftWing.kicad_sch)
- added sheet RightWing (p.kicad_sch)
- note added: "Put in a TFDU4301"

Commit message: Main schematic is done?
Parts:
- removed ?: (no value), symbol Device:LED
- removed J1: Conn_01x10_Female, symbol Connector:Conn_01x10_Female
- removed U1: QSE159, OptoDevice:ONSemi_QSE15x, symbol Interface_Optical:QSE159
- added ?: (no value), symbol Device:R
- added C11: .1uF, symbol Device:C
- added C12: 0.1uF, symbol Device:C
- added J2: Conn_01x14, symbol Connector_Generic:Conn_01x14
- added R3 (x2): R, symbol Device:R
- added U3: TFDU4301, symbol TFDU4301-IRDA:TFDU4301
Connections:
- net +3V3: now also R3.1, R3.1
- net +5V: now also J2.1 (Pin_1), J2.2 (Pin_2)
- net AMBIENT_LIGHT: now also ?.41 (GPIO29_ADC3), ?.2, C12.1; no longer ?.1, ?.2 (E)
- net CIPO: now also ?.6 (GPIO4)
- net COPI: now also ?.5 (GPIO3)
- net GND: now also C11.2, C12.2, J2.13 (Pin_13), J2.14 (Pin_14), U3.8 (GND)
- net MOTOR_A: now also ?.35 (GPIO23), ?.37 (GPIO25)
- net MOTOR_B: now also ?.36 (GPIO24)
- net NRF_CE: now also ?.8 (GPIO6)
- net NRF_CS: now also ?.7 (GPIO5)
- net NRF_IRQ: now also ?.9 (GPIO7)
- net SCK: now also ?.4 (GPIO2)
- net IRDA_SD: now reaches ?.11 (GPIO8)
- net IRDA_SD: now also U3.5 (SD)
- net IRDA_TX: now reaches ?.2 (GPIO0)
- net IRDA_TX: now also U3.3 (TXD)
- net SDA: now reaches ?.27 (GPIO16)
- net SDA: now also J2.7 (Pin_7)
- net SCL: now reaches ?.28 (GPIO17)
- net SCL: now also J2.8 (Pin_8)
- net IRDA_RX: now reaches ?.3 (GPIO1)
- net IRDA_RX: now also U3.4 (RXD)
- net PORT_LED_2: now reaches ?.30 (GPIO19)
- net PORT_LED_2: now also J2.4 (Pin_4)
- net PORT_LED_1: now reaches ?.31 (GPIO20)
- net PORT_LED_1: now also J2.3 (Pin_3)
- net STBD_LED_2: now reaches ?.32 (GPIO21)
- net STBD_LED_2: now also J2.6 (Pin_6)
- net STBD_LED_1: now reaches ?.34 (GPIO22)
- net STBD_LED_1: now also J2.5 (Pin_5)
- new net: C11.1, R3.2, U3.6 (VCC1)
- new net: ?.1, ?.1, ?.2 (E)
- new net: R3.2, U3.1 (VCC2_IRED-A)
- new net PORT_GP0: J2.9 (Pin_9)
- new net PORT_GP1: J2.10 (Pin_10)
- new net STBD_GP0: J2.11 (Pin_11)
- new net STBD_GP1: J2.12 (Pin_12)
- no-connect marks 0 -> 1
Other:
- sheet LeftWing renamed PortWing
- sheet RightWing renamed StbdWing
- sheet PortWing: file LeftWing.kicad_sch -> PortWing.kicad_sch
- sheet StbdWing: file p.kicad_sch -> StbdWing.kicad_sch
- note added: "This IRDA xcvr can be used to send AND receive remote control codes!!! See https://datasheet.octopart.com/TFBS4710-TT1-Vishay-datasheet-12514678.pdf"
- note removed: "Put in a TFDU4301"

Commit message: Schematic is done! Now to work on the main PCB
Parts:
- removed ? (x5): (no value), symbol Device:C
- removed ?: (no value), symbol Switch:SW_SPST
- removed ?: (no value), symbol Device:D_Schottky
- removed ?: (no value), symbol Device:Crystal
- removed C4 (x2), C8: C, symbol Device:C
- removed Y1: Crystal, symbol Device:Crystal
- added ? (x6): (no value), symbol Device:C
- added ?: (no value), symbol Device:D_Schottky
- added ?: (no value), symbol Device:R
- added C35 (x2), C4 (x3): C, symbol Device:C
- added D515 (x3): LED, symbol Device:LED
- added R20 (x3): 2.2K, Capacitor_SMD:C_0402_1005Metric, symbol Device:R
- added R6 (x2): R, symbol Device:R
- added R8 (x2): 27, symbol Device:R
- added SW3: SW_SPDT, Button_Switch_THT:SW_Push_1P2T_Vertical_E-Switch_800UDP8P1A1M6, symbol Switch:SW_SPDT
- added U25: AP3722AT, AP3722AT:AP3722AT, symbol AP3722AT-microphone:AP3722AT
- added Y3 (x2): Crystal_GND24_Small, Crystal:Crystal_SMD_3225-4Pin_3.2x2.5mm, symbol Device:Crystal_GND24_Small
- ?: LCSC (none) -> C497873
- ? (x7): now fitted
- ?: LCSC (none) -> C12891
- ?: LCSC (none) -> C318884
- ?: LCSC (none) -> C8678
- C1: LCSC (none) -> C1585
- C2: LCSC (none) -> C32949
- C4: LCSC (none) -> C1569
- C4: LSCS (none) -> C1531
- L1: LCSC (none) -> C27147
- L1: LCSC (none) -> C14033
- R1: LCSC (none) -> C25768
- U3: LCSC (none) -> C222418
Connections:
- net +3V3: now also ?.1, ?.2, C35.1, C4.1, U25.1 (VCC)
- net +5V: now also SW3.1 (A)
- net AMBIENT_LIGHT: now also ?.40 (GPIO28_ADC2); no longer ?.41 (GPIO29_ADC3)
- net GND: now also ?.2, ?.2, ?.2, ?.2, ?.2, C35.2, C35.2, C4.1, C4.2, C4.2, R20.2, R20.2, R6.2, U25.2 (GND), U25.3 (GND), Y3.2, Y3.2, Y3.4, Y3.4
- net HALL_SENSOR: now also ?.16 (GPIO13)
- net PORT_GP0: now also ?.15 (GPIO12)
- net PORT_GP1: now also ?.14 (GPIO11)
- net STBD_GP0: now also ?.13 (GPIO10)
- net STBD_GP1: now also ?.12 (GPIO9)
- net STBD_LED_1: now also ?.32 (GPIO21); no longer ?.34 (GPIO22)
- net STBD_LED_2: now also ?.18 (GPIO15); no longer ?.32 (GPIO21)
- net USB_D+: now also R8.1; no longer ?.46 (USB_DM)
- net USB_D-: now also R8.1; no longer ?.47 (USB_DP)
- net BATTERY_RAW: now reaches ?.1, ?.1 (+), ?.2 (VCC), ?.5 (BAT), ?.8 (FB)
- net BATTERY_RAW: now also ?.1, C35.1, R6.1
- net at ?.2, ?.5 (SW), ?.6 (SW)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: now also ?.2 (A)
- net at ?.1, ?.20 (XIN): now also Y3.1
- net VUSB: now reaches ?.2 (A), ?.4 (VIN), ?.A4 (VBUS), ?.A9 (VBUS), ?.B4 (VBUS), ?.B9 (VBUS)
- net VUSB: now also R20.2
- net at ?.11 (VDD_PA), C4.2, L1.1: now also C4.1
- net at ?.9 (XC2), C2.1, R2.2: now also Y3.3; no longer C2.1
- net at ?.1 (~{CS}), ?.2, ?.56 (QSPI_SS): now also ?.1
- net at ?.10 (XC1), R2.1: now also C2.1, Y3.1
- net at ?.1, ?.1, ?.1 (K): now also ?.1, ?.1 (K), SW3.2 (B)
- net at ?.17 (GPIO14): now also D515.2 (A)
- net at ?.1, ?.21 (XOUT): now also Y3.3
- net at ?.23 (DVDD), ?.50 (DVDD): now also ?.1
- net MIC_OUT: now reaches ?.38 (GPIO26_ADC0)
- net MIC_OUT: now also ?.2
- net at ?.39 (GPIO27_ADC1): now also R6.1, R6.2
- net at ?.4 (SS): now also ?.1
- net at AE1.1 (A), C4.2: now also C4.2
- net at ?.2 (ISET): now also R20.1
- net at ?.6 (DONE): now also D515.2 (A)
- net at ?.7 (CHRG): now also D515.2 (A)
- new net: D515.1 (K), D515.1 (K), R20.1
- new net: ?.47 (USB_DP), R8.2
- new net: D515.1 (K), R20.1
- new net: ?.46 (USB_DM), R8.2
- new net: ?.1, U25.4 (OUT)
Other:
- moved on the sheet: AE1, C1, C11, C12, C2, C4, C8, L1, R1, R2, R3, U3

Commit message: Hardware mods
Parts:
- removed AE1: Antenna, symbol Device:Antenna
- added AE2: Antenna_Chip, Resistor_SMD:R_1206_3216Metric, symbol Device:Antenna_Chip
- added J4: Conn_02x07_Odd_Even, symbol Connector_Generic:Conn_02x07_Odd_Even
- ?: Manufacturer PN CC6201ST -> (none)
- ?: LCSC C97521 -> (none)
- ?: LCSC C6186 -> (none)
- ?: Manufacturer PN Si24R1 -> (none)
- ?: LCSC C112011 -> (none)
- ?: LCSC C146233 -> (none)
- Y3: LCSC C9002 -> (none)
Connections:
- net USB_RES-: now reaches ?.47 (USB_DP), R8.2
- net at C4.2, C4.2: now also AE2.1 (FEED)
- net USB_RES+: now reaches ?.46 (USB_DM), R8.2
Other:
- moved on the sheet: R8

Commit message: Almost had the PCB done, need to restart. Sad face
Parts:
- removed AE2: Antenna_Chip, Resistor_SMD:R_1206_3216Metric, symbol Device:Antenna_Chip
- removed J2: Conn_01x14, symbol Connector_Generic:Conn_01x14
- added AE1: Antenna, RF_Antenna:Texas_SWRA117D_2.4GHz_Left, symbol Device:Antenna_Shield
- added BZ1: Buzzer, ButterflyBadge:Buzzer-GSC5025YA-12R4000, symbol Device:Buzzer
- added Q2: Q_NMOS_GSD, Package_TO_SOT_SMD:SOT-23, symbol Device:Q_NMOS_GSD
- added R23: 0, Resistor_SMD:R_0402_1005Metric, symbol Device:R
- added R24: 10K, Resistor_SMD:R_0402_1005Metric, symbol Device:R
- BT1: renamed from ?; value (none) -> Battery_Cell; footprint (none) -> Battery:BatteryHolder_MPD_BH-18650-PC2
- C1, C10, C13, C3, C33, C6: renamed from ?; value (none) -> 0.1uF; footprint (none) -> Capacitor_SMD:C_0402_1005Metric
- C11, C16, C29, C30, C31, C32, C34, C43, C5, C9: renamed from ?; value (none) -> 1uF; footprint (none) -> Capacitor_SMD:C_0402_1005Metric
- C15, C21, C44: renamed from ?; value (none) -> 22uF; footprint (none) -> Capacitor_SMD:C_1206_3216Metric
- C17: renamed from C8; value C -> 10nF; footprint (none) -> Capacitor_SMD:C_0402_1005Metric
- C18: renamed from C1; value C -> 33nF; footprint (none) -> Capacitor_SMD:C_0402_1005Metric
- C2, C4: renamed from ?; value (none) -> 20pF; footprint (none) -> Capacitor_SMD:C_0402_1005Metric
- C20: renamed from C12; footprint (none) -> Capacitor_SMD:C_0402_1005Metric
- C23, C46: renamed from C4; value C -> 2.2n; footprint (none) -> Capacitor_SMD:C_0402_1005Metric; LCSC (none) -> C1531
- C24, C41: renamed from C2; value C -> 9pF; footprint (none) -> Capacitor_SMD:C_0402_1005Metric
- C26: renamed from C11; footprint (none) -> Capacitor_SMD:C_0603_1608Metric
- C27, C28, C47: renamed from C4; value C -> 4.7pf; footprint (none) -> Capacitor_SMD:C_0402_1005Metric
- C42, C45: renamed from C35; value C -> 10uF; footprint (none) -> Capacitor_SMD:C_0603_1608Metric
- D1, D2: renamed from ?; value (none) -> D_Schottky; footprint (none) -> Diode_SMD:D_SMA
- D516, D517, D518: renamed from D515; footprint (none) -> LED_SMD:LED_0603_1608Metric
- J1: renamed from ?; value (none) -> USB_C_Receptacle_USB2.0; footprint (none) -> Connector_USB:USB_C_Receptacle_HRO_TYPE-C-31-M-12
- J4: footprint (none) -> ButterflyBadge:FlatFlexWingConnector-PCBSide
- L1: renamed from ?; value (none) -> 22uH; footprint (none) -> ButterflyBadge:YSPI0630A
- L2: renamed from L1; value L_Small -> 2.7nH; footprint (none) -> Inductor_SMD:L_0402_1005Metric
- L3: renamed from L1; value L_Small -> 8.2nH; footprint (none) -> Inductor_SMD:L_0402_1005Metric
- L4: renamed from L1; value L_Small -> 3.9nH; footprint (none) -> Inductor_SMD:L_0402_1005Metric
- M1: renamed from ?; value (none) -> Motor_DC; footprint (none) -> Connector_JST:JST_XH_B2B-XH-AM_1x02_P2.50mm_Vertical
- P1: renamed from ?; value (none) -> TC2030-CTX; footprint (none) -> Tag-Connect:TC2030-MCP-NL
- Q1: renamed from ?; value (none) -> ALS-PT19; footprint (none) -> Resistor_SMD:R_0402_1005Metric
- R1, R13, R16, R8: renamed from ?; value (none) -> 1K; footprint (none) -> Resistor_SMD:R_0402_1005Metric
- R10, R11: renamed from R6; value R -> 1K; footprint (none) -> Resistor_SMD:R_0402_1005Metric
- R12: renamed from ?; value (none) -> 4.22K; footprint (none) -> Resistor_SMD:R_0402_1005Metric
- R14: renamed from ?; value (none) -> 4.7K; footprint (none) -> Resistor_SMD:R_0402_1005Metric
- R15: renamed from R1; value R -> 22K; footprint (none) -> Resistor_SMD:R_0402_1005Metric
- R17, R18: renamed from R3; value R -> 0; footprint (none) -> Resistor_SMD:R_0402_1005Metric
- R19: renamed from R2; value R -> 1M; footprint (none) -> Resistor_SMD:R_0402_1005Metric
- R2, R3, R9: renamed from ?; value (none) -> 10K; footprint (none) -> Resistor_SMD:R_0402_1005Metric
- R21, R22: renamed from R20; value 2.2K -> 330
- R4, R5: renamed from ?; value (none) -> 5.1k; footprint (none) -> Resistor_SMD:R_0402_1005Metric
- R6, R7: renamed from R8; footprint (none) -> Resistor_SMD:R_0402_1005Metric
- SW1: renamed from ?; value (none) -> SW_Push; footprint (none) -> Button_Switch_SMD:SW_SPST_EVPBF
- U1: renamed from ?; value (none) -> W25Q128JVS; footprint (none) -> Package_SO:SOIC-8_5.23x5.23mm_P1.27mm
- U2: renamed from ?; value (none) -> CN3058; footprint (none) -> Package_SO:SOP-8_3.9x4.9mm_P1.27mm
- U3: renamed from ?; value (none) -> RP2040; footprint (none) -> Package_DFN_QFN:QFN-56-1EP_7x7mm_P0.4mm_EP3.2x3.2mm
- U4: renamed from ?; value (none) -> AX5201; footprint (none) -> Package_SO:SOIC-8-1EP_3.9x4.9mm_P1.27mm_EP2.41x3.3mm_ThermalVias
- U5: renamed from ?; value (none) -> AMS1117-3.3; footprint (none) -> Package_TO_SOT_SMD:SOT-223-3_TabPin2
- U6: renamed from ?; value (none) -> Si24R1; footprint (none) -> Package_DFN_QFN:QFN-20-1EP_4x4mm_P0.5mm_EP2.5x2.5mm
- U7: renamed from U3; footprint (none) -> TFDU4301:TFDU4301
- U8: renamed from ?; value (none) -> SM351LT; footprint (none) -> Package_TO_SOT_SMD:SOT-23
- U9: renamed from ?; value (none) -> TMI8118; footprint (none) -> Package_TO_SOT_SMD:SOT-23-6
- Y1: renamed from Y3; value Crystal_GND24_Small -> 12MHz
- Y2: renamed from Y3; value Crystal_GND24_Small -> 16MHz
Connections:
- net +5V: now also J4.1 (Pin_1), J4.2 (Pin_2), R23.1
- net GND: now also J4.13 (Pin_13), J4.14 (Pin_14), AE1.2 (Shield), Q2.2 (S), R24.2
- net PORT_GP0: now also J4.10 (Pin_10)
- net PORT_GP1: now also J4.12 (Pin_12)
- net PORT_LED_1: now also J4.4 (Pin_4)
- net PORT_LED_2: now also J4.6 (Pin_6)
- net SCL: now also J4.7 (Pin_7)
- net SDA: now also J4.8 (Pin_8)
- net STBD_GP0: now also J4.9 (Pin_9)
- net STBD_GP1: now also J4.11 (Pin_11)
- net STBD_LED_1: now also J4.3 (Pin_3)
- net STBD_LED_2: now also J4.5 (Pin_5)
- net at C27.2, C28.2: now also AE1.1 (A)
- new net: BZ1.1 (-), R23.2
- new net: BZ1.2 (+), Q2.3 (D)
- new net: Q2.1 (G), R24.1
Other:
- removed sheet PortWing
- removed sheet StbdWing
- moved on the sheet: J4
