File: Hardware/ButterflyBadge/ButterflyBadge.kicad_sch (KiCad schematic)
At the start: 90 parts, among them J1 USB_C_Receptacle_USB2.0, J4 Conn_02x07_Odd_Even, M1 Motor_DC, P1 TC2030-CTX, Q1 ALS-PT19, Q2 Q_NMOS_GSD, SW1 SW_Push, SW3 SW_SPDT, U1 W25Q128JVS, U2 CN3058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

Commit message: Component placement is done, now for layout
Parts:
- added C22, C25, C35: 22uF, Capacitor_SMD:C_1206_3216Metric, symbol Device:C
- added H1, H2, H3: (no value), MountingHole:MountingHole_3.2mm_M3, symbol Mechanical:MountingHole_Pad
- Q2: LCSC C15127 -> C8545
Connections:
- net +5V: now also C22.1, C25.1, C35.1
- net BUZZER: now also Q2.1 (G), R24.1, U3.29 (GPIO18)
- net GND: now also C22.2, C25.2, C35.2, H1.1, H2.1, H3.1
- net at C31.2, C32.1, U9.6 (OUTA): no longer M1.2 (-)
- net at C30.2, C31.1, U9.1 (OUTB): no longer M1.1 (+)
Other:
- moved on the sheet: M1

Commit message: Commit before I try to ripup everything on a whim
Connections:
- net BUZZER: no longer U3.29 (GPIO18)
- net CIPO: now also U3.31 (GPIO20); no longer U3.6 (GPIO4)
- net COPI: now also U3.30 (GPIO19); no longer U3.5 (GPIO3)
- net HALL_SENSOR: now also U3.41 (GPIO29_ADC3); no longer U3.16 (GPIO13)
- net MOTOR_A: no longer U3.35 (GPIO23)
- net NRF_CE: now also U3.34 (GPIO22); no longer U3.8 (GPIO6)
- net NRF_CS: now also U3.32 (GPIO21); no longer U3.7 (GPIO5)
- net NRF_IRQ: now also U3.35 (GPIO23); no longer U3.9 (GPIO7)
- net PORT_LED_1: no longer U3.31 (GPIO20)
- net PORT_LED_2: no longer U3.30 (GPIO19)
- net SCK: now also U3.29 (GPIO18); no longer U3.4 (GPIO2)
- net STBD_LED_1: no longer U3.32 (GPIO21)
Changed lines of the file:
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@@
+    (stroke (width 0) (type default))
+  )
+  (wire (pts (xy 146.05 105.41) (xy 151.13 105.41))
     (stroke (width 0) (type default))
   )
@@
     (stroke (width 0) (type default))
   )
+  (wire (pts (xy 146.05 110.49) (xy 154.94 110.49))
+    (stroke (width 0) (type default))
+  )
   (wire (pts (xy 234.95 209.55) (xy 234.95 212.09))
     (stroke (width 0) (type default))
@@
     (stroke (width 0) (type default))
   )
-  (wire (pts (xy 146.05 102.87) (xy 156.21 102.87))
-    (stroke (width 0) (type default))
-  )
   (wire (pts (xy 266.7 121.92) (xy 266.7 124.46))
     (stroke (width 0) (type default))
@@
     (stroke (width 0) (type default))
   )
+  (wire (pts (xy 146.05 102.87) (xy 149.86 102.87))
+    (stroke (width 0) (type default))
+  )
   (wire (pts (xy 71.12 240.03) (xy 71.12 231.14))
     (stroke (width 0) (type default))
@@
     (stroke (width 0) (type default))
   )
-  (wire (pts (xy 146.05 105.41) (xy 156.845 105.41))
-    (stroke (width 0) (type default))
-  )
   (wire (pts (xy 214.63 50.8) (xy 226.06 50.8))
     (stroke (width 0) (type default))
@@
     (stroke (width 0) (type default))
   )
+  (wire (pts (xy 146.05 107.95) (xy 151.13 107.95))
+    (stroke (width 0) (type default))
+  )
   (wire (pts (xy 369.57 213.36) (xy 369.57 215.9))
     (stroke (width 0) (type default))
@@
     (stroke (width 0) (type default))
   )
+  (wire (pts (xy 146.05 133.35) (xy 162.56 133.35))
+    (stroke (width 0) (type default))
+  )
   (wire (pts (xy 106.68 204.47) (xy 90.17 204.47))
     (stroke (width 0) (type default))
@@
     (stroke (width 0) (type default))
   )
-  (wire (pts (xy 146.05 110.49) (xy 156.21 110.49))
-    (stroke (width 0) (type default))
-  )
   (wire (pts (xy 118.11 49.53) (xy 118.11 23.495))
     (stroke (width 0) (type default))
@@
   )
   (wire (pts (xy 57.15 219.71) (xy 68.58 219.71))
-    (stroke (width 0) (type default))
-  )
-  (wire (pts (xy 146.05 107.95) (xy 156.845 107.95))
     (stroke (width 0) (type default))
   )
@@
     (effects (font (size 1.27 1.27)) (justify right bottom))
   )
-  (label "NRF_CS" (at 153.035 69.85 180) (fields_autoplaced)
+  (label "NRF_CS" (at 154.94 110.49 180) (fields_autoplaced)
     (effects (font (size 1.27 1.27)) (justify right bottom))
   )
@@
     (effects (font (size 1.27 1.27)) (justify left bottom))
   )
-  (label "CIPO" (at 147.955 67.31 0) (fields_autoplaced)
-    (effects (font (size 1.27 1.27)) (justify left bottom))
+  (label "CIPO" (at 151.13 107.95 180) (fields_autoplaced)
+    (effects (font (size 1.27 1.27)) (justify right bottom))
   )
   (label "MOTOR_A" (at 155.575 120.65 180) (fields_autoplaced)
@@
     (effects (font (size 1.27 1.27)) (justify left bottom))
   )
-  (label "BUZZER" (at 148.59 102.87 0) (fields_autoplaced)
+  (label "BUZZER" (at 179.07 71.12 0) (fields_autoplaced)
     (effects (font (size 1.27 1.27)) (justify left bottom))
   )
@@
     (effects (font (size 1.27 1.27)) (justify left bottom))
   )
-  (label "MOTOR_A" (at 155.575 115.57 180) (fields_autoplaced)
+  (label "MOTOR_A" (at 176.53 105.41 180) (fields_autoplaced)
     (effects (font (size 1.27 1.27)) (justify right bottom))
   )
@@
     (effects (font (size 1.27 1.27)) (justify left bottom))
   )
-  (label "COPI" (at 147.955 64.77 0) (fields_autoplaced)
-    (effects (font (size 1.27 1.27)) (justify left bottom))
+  (label "COPI" (at 151.13 105.41 180) (fields_autoplaced)
+    (effects (font (size 1.27 1.27)) (justify right bottom))
   )
   (label "STBD_LED_2" (at 158.75 95.25 180) (fields_autoplaced)
@@
     (effects (font (size 1.27 1.27)) (justify left bottom))
   )
-  (label "NRF_IRQ" (at 146.05 74.93 0) (fields_autoplaced)
-    (effects (font (size 1.27 1.27)) (justify left bottom))
+  (label "NRF_IRQ" (at 154.94 115.57 180) (fields_autoplaced)
+    (effects (font (size 1.27 1.27)) (justify right bottom))
   )
   (label "USB_RES-" (at 85.09 64.77 0) (fields_autoplaced)
@@
     (effects (font (size 1.27 1.27)) (justify left bottom))
   )
-  (label "SCK" (at 147.955 62.23 0) (fields_autoplaced)
-    (effects (font (size 1.27 1.27)) (justify left bottom))
+  (label "SCK" (at 149.86 102.87 180) (fields_autoplaced)
+    (effects (font (size 1.27 1.27)) (justify right bottom))
   )
   (label "RST" (at 47.625 132.08 0) (fields_autoplaced)
@@
     (effects (font (size 1.27 1.27)) (justify right bottom))
   )
-  (label "NRF_CE" (at 151.765 72.39 180) (fields_autoplaced)
+  (label "NRF_CE" (at 156.21 113.03 180) (fields_autoplaced)
     (effects (font (size 1.27 1.27)) (justify right bottom))
   )
@@
     (effects (font (size 1.27 1.27)) (justify left bottom))
   )
-  (label "STBD_LED_1" (at 156.21 110.49 180) (fields_autoplaced)
-    (effects (font (size 1.27 1.27)) (justify right bottom))
-  )
-  (label "HALL_SENSOR" (at 160.02 90.17 180) (fields_autoplaced)
-    (effects (font (size 1.27 1.27)) (justify right bottom))
-  )
-  (label "PORT_LED_2" (at 156.845 105.41 180) (fields_autoplaced)
+  (label "STBD_LED_1" (at 186.69 78.74 180) (fields_autoplaced)
+    (effects (font (size 1.27 1.27)) (justify right bottom))
+  )
+  (label "HALL_SENSOR" (at 162.56 133.35 180) (fields_autoplaced)
+    (effects (font (size 1.27 1.27)) (justify right bottom))
+  )
+  (label "PORT_LED_2" (at 187.325 73.66 180) (fields_autoplaced)
     (effects (font (size 1.27 1.27)) (justify right bottom))
   )
@@
     (effects (font (size 1.27 1.27)) (justify right bottom))
   )
-  (label "PORT_LED_1" (at 156.845 107.95 180) (fields_autoplaced)
-    (effects (font (size 1.27 1.27)) (justify right bottom))
-  )
+  (label "PORT_LED_1" (at 187.325 76.2 180) (fields_autoplaced)
+    (effects (font (size 1.27 1.27)) (justify right bottom))
+  )

Commit message: More routing
Parts:
- removed C3: 0.1uF, Capacitor_SMD:C_0402_1005Metric, symbol Device:C
- added TP1, TP2, TP3: (no value), TestPoint:TestPoint_Pad_D1.0mm, symbol Connector:TestPoint
Connections:
- net BUZZER: now also U3.38 (GPIO26_ADC0)
- net CIPO: now also U3.11 (GPIO8); no longer U3.31 (GPIO20)
- net COPI: now also U3.9 (GPIO7); no longer U3.30 (GPIO19)
- net GND: now also U6.21 (EP)
- net HALL_SENSOR: now also U3.5 (GPIO3); no longer U3.41 (GPIO29_ADC3)
- net IRDA_SD: now also U3.4 (GPIO2); no longer U3.11 (GPIO8)
- net MIC_OUT: now also U3.41 (GPIO29_ADC3); no longer U3.38 (GPIO26_ADC0)
- net MOTOR_A: now also U3.14 (GPIO11); no longer U3.37 (GPIO25)
- net MOTOR_B: now also U3.13 (GPIO10); no longer U3.36 (GPIO24)
- net NRF_CE: now also U3.6 (GPIO4); no longer U3.34 (GPIO22)
- net NRF_CS: now also U3.7 (GPIO5); no longer U3.32 (GPIO21)
- net NRF_IRQ: now also U3.12 (GPIO9); no longer U3.35 (GPIO23)
- net PORT_GP0: now also U3.18 (GPIO15); no longer U3.15 (GPIO12)
- net PORT_GP1: now also U3.16 (GPIO13); no longer U3.14 (GPIO11)
- net PORT_LED_1: now also U3.32 (GPIO21)
- net PORT_LED_2: now also U3.30 (GPIO19)
- net SCK: now also U3.8 (GPIO6); no longer U3.29 (GPIO18)
- net STBD_GP0: now also U3.17 (GPIO14); no longer U3.13 (GPIO10)
- net STBD_GP1: now also U3.15 (GPIO12); no longer U3.12 (GPIO9)
- net STBD_LED_1: now also U3.31 (GPIO20)
- net STBD_LED_2: now also U3.29 (GPIO18); no longer U3.18 (GPIO15)
- net at C31.2, C32.1, U9.6 (OUTA): now also M1.2 (-)
- net at M1.1 (+): now also C30.2, C31.1, U9.1 (OUTB)
- net 5V_UNSWITCHED: now reaches C16.1, C21.1, D1.1 (K), D2.1 (K), R12.1, SW3.2 (B)
- net LED: now reaches D518.2 (A)
- net LED: now also U3.34 (GPIO22); no longer U3.17 (GPIO14)
- new net: TP2.1, U3.36 (GPIO24)
- new net: TP1.1, U3.35 (GPIO23)
- new net: TP3.1, U3.37 (GPIO25)
Other:
- moved on the sheet: D518, M1, R22

Commit message: Commit before changing board outline
Parts:
- removed H1, H2, H3: (no value), MountingHole:MountingHole_3.2mm_M3, symbol Mechanical:MountingHole_Pad
Changed lines of the file:
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@@
     )
   )
-  (symbol (lib_id "Mechanical:MountingHole_Pad") (at 46.99 152.4 0) (unit 1)
-    (in_bom yes) (on_board yes) (dnp no) (fields_autoplaced)
-    (property "Reference" "H2" (at 49.53 150.495 0)
-      (effects (font (size 1.27 1.27)) (justify left))
-    )
-    (property "Value" " " (at 49.53 153.035 0)
-      (effects (font (size 1.27 1.27)) (justify left))
-    )
-    (property "Footprint" "MountingHole:MountingHole_3.2mm_M3" (at 46.99 152.4 0)
-      (effects (font (size 1.27 1.27)) hide)
-    )
-    (property "Datasheet" "~" (at 46.99 152.4 0)
-      (effects (font (size 1.27 1.27)) hide)
-    )
-    (property "Manufacturer PN" "" (at 46.99 152.4 0)
-      (effects (font (size 1.27 1.27)))
-    )
-    (pin "1")
-    (instances
-      (project "ButterflyBadge"
-        (path "/0dfc5389-1533-4aa5-854f-8445ef0ba5aa"
-          (reference "H2") (unit 1) (value " ") (footprint "MountingHole:MountingHole_3.2mm_M3")
-        )
-      )
-    )
-  )
   (symbol (lib_id "Device:L_Small") (at 163.83 224.79 90) (unit 1)
     (in_bom yes) (on_board yes) (dnp no)
@@
     )
   )
-  (symbol (lib_id "Mechanical:MountingHole_Pad") (at 54.61 152.4 0) (unit 1)
-    (in_bom yes) (on_board yes) (dnp no) (fields_autoplaced)
-    (property "Reference" "H3" (at 57.15 150.495 0)
-      (effects (font (size 1.27 1.27)) (justify left))
-    )
-    (property "Value" " " (at 57.15 153.035 0)
-      (effects (font (size 1.27 1.27)) (justify left))
-    )
-    (property "Footprint" "MountingHole:MountingHole_3.2mm_M3" (at 54.61 152.4 0)
-      (effects (font (size 1.27 1.27)) hide)
-    )
-    (property "Datasheet" "~" (at 54.61 152.4 0)
-      (effects (font (size 1.27 1.27)) hide)
-    )
-    (property "Manufacturer PN" "" (at 54.61 152.4 0)
-      (effects (font (size 1.27 1.27)))
-    )
-    (pin "1")
-    (instances
-      (project "ButterflyBadge"
-        (path "/0dfc5389-1533-4aa5-854f-8445ef0ba5aa"
-          (reference "H3") (unit 1) (value " ") (footprint "MountingHole:MountingHole_3.2mm_M3")
-        )
-      )
-    )
-  )
   (symbol (lib_id "Device:C") (at 76.835 106.68 0) (unit 1)
     (in_bom yes) (on_board yes) (dnp no) (fields_autoplaced)
@@
     )
   )
-  (symbol (lib_id "power:GND") (at 39.37 154.94 0) (unit 1)
-    (in_bom yes) (on_board yes) (dnp no) (fields_autoplaced)
-    (property "Reference" "#PWR0190" (at 39.37 161.29 0)
-      (effects (font (size 1.27 1.27)) hide)
-    )
-    (property "Value" "GND" (at 39.37 160.02 0)
-      (effects (font (size 1.27 1.27)))
-    )
-    (property "Footprint" "" (at 39.37 154.94 0)
-      (effects (font (size 1.27 1.27)) hide)
-    )
-    (property "Datasheet" "" (at 39.37 154.94 0)
-      (effects (font (size 1.27 1.27)) hide)
-    )
-    (pin "1")
-    (instances
-      (project "ButterflyBadge"
-        (path "/0dfc5389-1533-4aa5-854f-8445ef0ba5aa"
-          (reference "#PWR0190") (unit 1) (value "GND") (footprint "")
-        )
-      )
-    )
-  )
   (symbol (lib_id "power:GND") (at 344.17 195.58 0) (unit 1)
     (in_bom yes) (on_board yes) (dnp no) (fields_autoplaced)
@@
     )
   )
-  (symbol (lib_id "power:GND") (at 46.99 154.94 0) (unit 1)
-    (in_bom yes) (on_board yes) (dnp no) (fields_autoplaced)
-    (property "Reference" "#PWR0194" (at 46.99 161.29 0)
-      (effects (font (size 1.27 1.27)) hide)
-    )
-    (property "Value" "GND" (at 46.99 160.02 0)
-      (effects (font (size 1.27 1.27)))
-    )
-    (property "Footprint" "" (at 46.99 154.94 0)
-      (effects (font (size 1.27 1.27)) hide)
-    )
-    (property "Datasheet" "" (at 46.99 154.94 0)
-      (effects (font (size 1.27 1.27)) hide)
-    )
-    (pin "1")
-    (instances
-      (project "ButterflyBadge"
-        (path "/0dfc5389-1533-4aa5-854f-8445ef0ba5aa"
-          (reference "#PWR0194") (unit 1) (value "GND") (footprint "")
-        )
-      )
-    )
-  )
   (symbol (lib_id "Ax5201:AX5201") (at 162.56 245.11 0) (unit 1)
     (in_bom yes) (on_board yes) (dnp no)
@@
         )
       )
-    )
-  )
-  (symbol (lib_id "power:GND") (at 54.61 154.94 0) (unit 1)
-    (in_bom yes) (on_board yes) (dnp no) (fields_autoplaced)
-    (property "Reference" "#PWR0191" (at 54.61 161.29 0)
-      (effects (font (size 1.27 1.27)) hide)
-    )
-    (property "Value" "GND" (at 54.61 160.02 0)
-      (effects (font (size 1.27 1.27)))
-    )
-    (property "Footprint" "" (at 54.61 154.94 0)
-      (effects (font (size 1.27 1.27)) hide)
-    )
-    (property "Datasheet" "" (at 54.61 154.94 0)
-      (effects (font (size 1.27 1.27)) hide)
-    )
-    (pin "1")
-    (instances
-      (project "ButterflyBadge"
-        (path "/0dfc5389-1533-4aa5-854f-8445ef0ba5aa"
-          (reference "#PWR0191") (unit 1) (value "GND") (footprint "")
-        )
-      )
-    )
-  )
-  (symbol (lib_id "Mechanical:MountingHole_Pad") (at 39.37 152.4 0) (unit 1)
-    (in_bom yes) (on_board yes) (dnp no) (fields_autoplaced)
-    (property "Reference" "H1" (at 41.91 150.495 0)
-      (effects (font (size 1.27 1.27)) (justify left))
-    )
-    (property "Value" " " (at 41.91 153.035 0)
-      (effects (font (size 1.27 1.27)) (justify left))
-    )
-    (property "Footprint" "MountingHole:MountingHole_3.2mm_M3" (at 39.37 152.4 0)
-      (effects (font (size 1.27 1.27)) hide)
-    )
-    (property "Datasheet" "~" (at 39.37 152.4 0)
-      (effects (font (size 1.27 1.27)) hide)
-    )
-    (property "Manufacturer PN" "" (at 39.37 152.4 0)
-      (effects (font (size 1.27 1.27)))
-    )
-    (pin "1")
-    (instances
-      (project "ButterflyBadge"
-        (path "/0dfc5389-1533-4aa5-854f-8445ef0ba5aa"
-          (reference "H1") (unit 1) (value " ") (footprint "MountingHole:MountingHole_3.2mm_M3")
-        )
-      )
