File: Hardware/PortWing/PortWing.kicad_sch (KiCad schematic)
At the start: 266 parts, among them J4 Conn_01x08, U1 XC6206PxxxMR, U5 SN74LV1T34DBV, X1 Badgelife_sao_connector_v169b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

Commit message: Started the port wing, was able to pull locations from starboard
Parts:
- removed C35 (x2): C, symbol Device:C
- removed J4: Conn_01x08, symbol Connector_Generic:Conn_01x08
- removed U1: XC6206PxxxMR, Package_TO_SOT_SMD:SOT-23, symbol Regulator_Linear:XC6206PxxxMR
- removed X1: Badgelife_sao_connector_v169bis, badgelife_sao_v169bis:Badgelife-SAOv169-BADGE-2x3, symbol badgelife_shitty_addon_v169bis:Badgelife_sao_connector_v169bis
- added C38 (x6): 22uF, Capacitor_SMD:C_1206_3216Metric, symbol Device:C
- added C39 (x3): 10uF, Capacitor_SMD:C_0603_1608Metric, symbol Device:C
- added J1: Conn_02x04_Odd_Even, ButterflyBadge:FlatFlexWingConnector-WingPCBSide, symbol Connector_Generic:Conn_02x04_Odd_Even
- added J14: Conn_02x06_Counter_Clockwise, Package_DIP:DIP-12_W10.16mm_LongPads, symbol Connector_Generic:Conn_02x06_Counter_Clockwise
- added U21: XC6206PxxxMR, Package_TO_SOT_SMD:SOT-23, symbol Regulator_Linear:XC6206PxxxMR
- added X2: Badgelife_sao_connector_v169bis, badgelife_sao_v169bis:Badgelife-SAOv169-BADGE-2x3, symbol badgelife_shitty_addon_v169bis:Badgelife_sao_connector_v169bis
- C37: renamed from C35; value C -> 1uF; footprint (none) -> Capacitor_SMD:C_0402_1005Metric
- U15: renamed from ?; value (none) -> ~
- U16: renamed from ?; value (none) -> ~; footprint (none) -> Package_SO:SOP-8_3.9x4.9mm_P1.27mm
- renumbered D2 to D10, D2 to D100, D2 to D101, D2 to D102, D2 to D103, D2 to D104, D2 to D105, D2 to D106, D2 to D107, D2 to D108, D2 to D109, D2 to D11, D2 to D110, D2 to D111, D2 to D112, D2 to D113, D2 to D114, D2 to D115, D2 to D116, D2 to D117, D2 to D118, D2 to D119, D2 to D12, D2 to D120, D2 to D121, D2 to D122, D2 to D123, D2 to D124, D2 to D125, D2 to D126, D2 to D127, D2 to D128, D2 to D129, D2 to D13, D2 to D130, D2 to D131, D2 to D132, D2 to D133, D2 to D134, D2 to D135, D2 to D136, D2 to D137, D2 to D138, D2 to D139, D2 to D14, D2 to D140, D2 to D141, D2 to D142, D2 to D143, D2 to D144, D2 to D145, D2 to D146, D2 to D147, D2 to D148, D2 to D149, D2 to D15, D2 to D150, D2 to D151, D2 to D152, D2 to D153, D2 to D154, D2 to D155, D2 to D156, D2 to D157, D2 to D158, D2 to D159, D2 to D16, D2 to D160, D2 to D161, D2 to D162, D2 to D163, D2 to D164, D2 to D165, D2 to D166, D2 to D167, D2 to D168, D2 to D169, D2 to D17, D2 to D170, D2 to D171, D2 to D172, D2 to D173, D2 to D174, D2 to D175, D2 to D176, D2 to D177, D2 to D178, D2 to D179, D2 to D18, D2 to D180, D2 to D181, D2 to D182, D2 to D183, D2 to D184, D2 to D185, D2 to D186, D2 to D187, D2 to D188, D2 to D189, D2 to D19, D2 to D190, D2 to D191, D2 to D192, D2 to D193, D2 to D194, D2 to D195, D2 to D196, D2 to D197, D2 to D198, D2 to D199, D2 to D20, D2 to D200, D2 to D201, D2 to D202, D2 to D203, D2 to D204, D2 to D205, D2 to D206, D2 to D207, D2 to D208, D2 to D209, D2 to D21, D2 to D210, D2 to D211, D2 to D212, D2 to D213, D2 to D214, D2 to D215, D2 to D216, D2 to D217, D2 to D218, D2 to D219, D2 to D22, D2 to D220, D2 to D221, D2 to D222, D2 to D223, D2 to D224, D2 to D225, D2 to D226, D2 to D227, D2 to D228, D2 to D229, D2 to D23, D2 to D230, D2 to D231, D2 to D232, D2 to D233, D2 to D234, D2 to D235, D2 to D236, D2 to D237, D2 to D238, D2 to D239, D2 to D24, D2 to D240, D2 to D241, D2 to D242, D2 to D243, D2 to D244, D2 to D245, D2 to D246, D2 to D247, D2 to D248, D2 to D249, D2 to D25, D2 to D250, D2 to D251, D2 to D252, D2 to D253, D2 to D254, D2 to D255, D2 to D256, D2 to D257, D2 to D258, D2 to D26, D2 to D27, D2 to D28, D2 to D29, D2 to D3, D2 to D30, D2 to D31, D2 to D32, D2 to D33, D2 to D34, D2 to D35, D2 to D36, D2 to D37, D2 to D38, D2 to D39, D2 to D4, D2 to D40, D2 to D41, D2 to D42, D2 to D43, D2 to D44, D2 to D45, D2 to D46, D2 to D47, D2 to D48, D2 to D49, D2 to D5, D2 to D50, D2 to D51, D2 to D52, D2 to D53, D2 to D54, D2 to D55, D2 to D56, D2 to D57, D2 to D58, D2 to D59, D2 to D6, D2 to D60, D2 to D61, D2 to D62, D2 to D63, D2 to D64, D2 to D65, D2 to D66, D2 to D67, D2 to D68, D2 to D69, D2 to D7, D2 to D70, D2 to D71, D2 to D72, D2 to D73, D2 to D74, D2 to D75, D2 to D76, D2 to D77, D2 to D78, D2 to D79, D2 to D8, D2 to D80, D2 to D81, D2 to D82, D2 to D83, D2 to D84, D2 to D85, D2 to D86, D2 to D87, D2 to D88, D2 to D89, D2 to D9, D2 to D90, D2 to D91, D2 to D92, D2 to D93, D2 to D94, D2 to D95, D2 to D96, D2 to D97, D2 to D98, D2 to D99, U5 to U11, U5 to U12
Connections:
- net 3V3: now also C39.1, C39.1, C39.1, U21.2 (VO), X2.1 (VCC)
- net 5V: now also C38.1, C38.1, C38.1, C38.1, C38.1, C38.1, J1.1 (Pin_1), U21.3 (VI)
- net GND: now also C38.2, C38.2, C38.2, C38.2, C38.2, C38.2, C39.2, C39.2, C39.2, J1.3 (Pin_3), U21.1 (GND), X2.2 (GND)
- net NFC_MSG: now also J1.8 (Pin_8), X2.6 (GPIO2)
- net PORT_GP0: now also J1.6 (Pin_6), X2.5 (GPIO1)
- net PORT_LED_1: now also J1.2 (Pin_2)
- net PORT_LED_2: now also J1.4 (Pin_4)
- net SCL: now also J1.5 (Pin_5), X2.4 (SCL)
- net SDA: now also J1.7 (Pin_7), X2.3 (SDA)

Commit message: Re-moved everything
Parts:
- removed U15: ~, symbol Device:Antenna_Loop
- added JP1: Jumper_3_Bridged12, Jumper:SolderJumper-3_P1.3mm_Bridged12_Pad1.0x1.5mm, symbol Jumper:Jumper_3_Bridged12
Connections:
- net ANTENNA: now reaches U16.2 (AC0)
- net ANTENNA: now also U16.3 (AC1)
- net at U12.4 (Y): now also JP1.1 (A); no longer D11.2 (DIN)
- net PORT_LED1_OUT: now reaches D250.4 (DOUT)
- net PORT_LED1_OUT: now also JP1.3 (B)
- new net: D11.2 (DIN), JP1.2 (C)
Other:
- moved on the sheet: J14
Changed lines of the file:
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@@
     (stroke (width 0) (type default))
   )
+  (wire (pts (xy 101.6 370.84) (xy 101.6 364.49))
+    (stroke (width 0) (type default))
+  )
   (wire (pts (xy 135.89 53.34) (xy 135.89 58.42))
     (stroke (width 0) (type default))
@@
     (stroke (width 0) (type default))
   )
+  (wire (pts (xy 127 43.18) (xy 125.73 43.18))
+    (stroke (width 0) (type default))
+  )
   (wire (pts (xy 138.43 34.29) (xy 138.43 30.48))
     (stroke (width 0) (type default))
   )
-  (wire (pts (xy 92.71 370.84) (xy 105.41 370.84))
+  (wire (pts (xy 105.41 370.84) (xy 101.6 370.84))
+    (stroke (width 0) (type default))
+  )
+  (wire (pts (xy 92.71 370.84) (xy 93.98 370.84))
     (stroke (width 0) (type default))
   )
@@
     (stroke (width 0) (type default))
   )
+  (wire (pts (xy 125.73 45.72) (xy 127 45.72))
+    (stroke (width 0) (type default))
+  )
   (wire (pts (xy 346.71 271.78) (xy 95.25 271.78))
     (stroke (width 0) (type default))
@@
     (stroke (width 0) (type default))
   )
+  (wire (pts (xy 101.6 364.49) (xy 97.79 364.49))
+    (stroke (width 0) (type default))
+  )
   (wire (pts (xy 105.41 529.59) (xy 100.33 529.59))
     (stroke (width 0) (type default))
@@
     (stroke (width 0) (type default))
   )
+  (wire (pts (xy 125.73 43.18) (xy 125.73 45.72))
+    (stroke (width 0) (type default))
+  )
   (wire (pts (xy 101.6 464.82) (xy 101.6 476.25))
     (stroke (width 0) (type default))
@@
     (effects (font (size 1.27 1.27)) (justify right bottom))
   )
+  (label "PORT_LED1_OUT" (at 342.9 337.82 0) (fields_autoplaced)
+    (effects (font (size 1.27 1.27)) (justify left bottom))
+  )
   (label "5V" (at 289.56 330.2 90) (fields_autoplaced)
     (effects (font (size 1.27 1.27)) (justify left bottom))
@@
     (effects (font (size 1.27 1.27)) (justify right bottom))
   )
+  (label "PORT_LED1_OUT" (at 93.98 358.14 0) (fields_autoplaced)
+    (effects (font (size 1.27 1.27)) (justify left bottom))
+  )
   (label "5V" (at 137.16 302.26 90) (fields_autoplaced)
     (effects (font (size 1.27 1.27)) (justify left bottom))
@@
     (effects (font (size 1.27 1.27)) (justify left bottom))
   )
+  (label "ANTENNA" (at 125.73 43.18 180) (fields_autoplaced)
+    (effects (font (size 1.27 1.27)) (justify right bottom))
+  )
   (label "5V" (at 335.28 276.86 90) (fields_autoplaced)
     (effects (font (size 1.27 1.27)) (justify left bottom))
@@
       (effects (font (size 1.27 1.27)) hide)
     )
+    (property "Manufacturer PN" "" (at 78.74 151.13 0)
+      (effects (font (size 1.27 1.27)))
+    )
     (pin "1")
     (pin "2")
@@
       (project "PortWing"
         (path "/926ace71-90a7-4e38-a3e6-a8d44ceefc3f"
-          (reference "U4") (unit 1) (value "SN74LV1T34DBV") (footprint "Package_TO_SOT_SMD:SOT-23-5")
+          (reference "U3") (unit 1) (value "SN74LV1T34DBV") (footprint "Package_TO_SOT_SMD:SOT-23-5")
         )
       )
@@
     )
   )
-  (symbol (lib_id "Device:Antenna_Loop") (at 121.92 45.72 90) (unit 1)
-    (in_bom yes) (on_board yes) (dnp no) (fields_autoplaced)
-    (property "Reference" "U15" (at 121.92 35.56 90)
-      (effects (font (size 1.27 1.27)))
-    )
-    (property "Value" "~" (at 121.92 38.1 90)
-      (effects (font (size 1.27 1.27)))
-    )
-    (property "Footprint" "" (at 121.92 45.72 0)
-      (effects (font (size 1.27 1.27)) hide)
-    )
-    (property "Datasheet" "~" (at 121.92 45.72 0)
-      (effects (font (size 1.27 1.27)) hide)
-    )
-    (pin "1")
-    (pin "2")
-    (instances
-      (project "ButterflyBadge"
-        (path "/0dfc5389-1533-4aa5-854f-8445ef0ba5aa/e6b4de02-28de-4ad7-98dc-630452296216"
-          (reference "U15") (unit 1) (value "~") (footprint "")
-        )
-      )
-      (project "PortWing"
-        (path "/926ace71-90a7-4e38-a3e6-a8d44ceefc3f"
-          (reference "U3") (unit 1) (value "~") (footprint "")
-        )
-      )
-    )
-  )
   (symbol (lib_id "LED:SK6812") (at 335.28 204.47 0) (unit 1)
     (in_bom yes) (on_board yes) (dnp no)
@@
       (effects (font (size 1.27 1.27)) hide)
     )
+    (property "Manufacturer PN" "" (at 85.09 370.84 0)
+      (effects (font (size 1.27 1.27)))
+    )
     (pin "1")
     (pin "2")
@@
       (project "PortWing"
         (path "/926ace71-90a7-4e38-a3e6-a8d44ceefc3f"
-          (reference "U5") (unit 1) (value "SN74LV1T34DBV") (footprint "Package_TO_SOT_SMD:SOT-23-5")
+          (reference "U4") (unit 1) (value "SN74LV1T34DBV") (footprint "Package_TO_SOT_SMD:SOT-23-5")
         )
       )
@@
     )
   )
+  (symbol (lib_id "Jumper:Jumper_3_Bridged12") (at 93.98 364.49 90) (unit 1)
+    (in_bom yes) (on_board yes) (dnp no) (fields_autoplaced)
+    (property "Reference" "JP1" (at 91.44 363.855 90)
+      (effects (font (size 1.27 1.27)) (justify left))
+    )
+    (property "Value" "Jumper_3_Bridged12" (at 91.44 366.395 90)
+      (effects (font (size 1.27 1.27)) (justify left))
+    )
+    (property "Footprint" "Jumper:SolderJumper-3_P1.3mm_Bridged12_Pad1.0x1.5mm" (at 93.98 364.49 0)
+      (effects (font (size 1.27 1.27)) hide)
+    )
+    (property "Datasheet" "~" (at 93.98 364.49 0)
+      (effects (font (size 1.27 1.27)) hide)
+    )
+    (property "Manufacturer PN" "" (at 93.98 364.49 0)
+      (effects (font (size 1.27 1.27)))
+    )
+    (pin "1")
+    (pin "2")
+    (pin "3")
+    (instances
+      (project "PortWing"
+        (path "/926ace71-90a7-4e38-a3e6-a8d44ceefc3f"
+          (reference "JP1") (unit 1) (value "Jumper_3_Bridged12") (footprint "Jumper:SolderJumper-3_P1.3mm_Bridged12_Pad1.0x1.5mm")
+        )
+      )
+    )
+  )
   (symbol (lib_id "LED:SK6812") (at 265.43 476.25 0) (unit 1)
     (in_bom yes) (on_board yes) (dnp no)
@@
     )
   )
-  (symbol (lib_id "Connector_Generic:Conn_02x06_Counter_Clockwise") (at 309.88 97.79 0) (unit 1)
+  (symbol (lib_id "Connector_Generic:Conn_02x06_Counter_Clockwise") (at 111.76 111.76 0) (unit 1)
     (in_bom yes) (on_board yes) (dnp no) (fields_autoplaced)
-    (property "Reference" "J14" (at 311.15 87.63 0)
+    (property "Reference" "J14" (at 113.03 101.6 0)
       (effects (font (size 1.27 1.27)))
     )
-    (property "Value" "Conn_02x06_Counter_Clockwise" (at 311.15 90.17 0)
+    (property "Value" "Conn_02x06_Counter_Clockwise" (at 113.03 104.14 0)
       (effects (font (size 1.27 1.27)))
     )
-    (property "Footprint" "Package_DIP:DIP-12_W10.16mm_LongPads" (at 309.88 97.79 0)
+    (property "Footprint" "Package_DIP:DIP-12_W10.16mm_LongPads" (at 111.76 111.76 0)
       (effects (font (size 1.27 1.27)) hide)
     )
-    (property "Datasheet" "~" (at 309.88 97.79 0)
+    (property "Datasheet" "~" (at 111.76 111.76 0)
       (effects (font (size 1.27 1.27)) hide)
     )
-    (property "Manufacturer PN" "" (at 309.88 97.79 0)
+    (property "Manufacturer PN" "" (at 111.76 111.76 0)
       (effects (font (size 1.27 1.27)))
     )
@@
       (project "PortWing"
         (path "/926ace71-90a7-4e38-a3e6-a8d44ceefc3f"
-          (reference "J2") (unit 1) (value "Conn_02x06_Counter_Clockwise") (footprint "Package_DIP:DIP-12_W10.16mm_LongPads")
+          (reference "J14") (unit 1) (value "Conn_02x06_Counter_Clockwise") (footprint "Package_DIP:DIP-12_W10.16mm_LongPads")
         )
       )
@@
       (effects (font (size 1.27 1.27)) (justify left))
     )
+    (property "Manufacturer PN" "" (at 135.89 44.45 0)
+      (effects (font (size 1.27 1.27)))
+    )
     (pin "1")
