File: Hardware/StarboardWing/StarboardWing.kicad_sch (KiCad schematic)
At the start: 285 parts, among them J1 Conn_02x04_Odd_Even, J14 Conn_02x06_Counter_Clockwise, J7 Conn_01x01_Female, U19 SN74LV1T34DBV, U20 SN74LV1T34DBV, U21 XC6206PxxxMR, U23 HX612, X2 Badgelife_sao_connector_v169b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

Commit message: Re-moved everything
Parts:
- removed JP1: Jumper_2_Open, Jumper:SolderJumper-2_P1.3mm_Open_Pad1.0x1.5mm, symbol Jumper:Jumper_2_Open
- added JP1: Jumper_3_Bridged12, Jumper:SolderJumper-3_P1.3mm_Bridged12_Pad1.0x1.5mm, symbol Jumper:Jumper_3_Bridged12
Connections:
- net STBD_LED_1_OUT: now also JP1.3 (B)
- net at U23.1 (CH8): no longer J7.1 (Pin_1)
- net at U23.10 (CH1): now also J7.1 (Pin_1); no longer J7.1 (Pin_1)
- net at U23.11 (CH2): now also J7.1 (Pin_1); no longer J7.1 (Pin_1)
- net at U23.12 (CH3): now also J7.1 (Pin_1); no longer J7.1 (Pin_1)
- net at U23.13 (CH4): now also J7.1 (Pin_1); no longer J7.1 (Pin_1)
- net at U23.14 (CH5): now also J7.1 (Pin_1); no longer J7.1 (Pin_1)
- net at U23.15 (CH6): now also J7.1 (Pin_1); no longer J7.1 (Pin_1)
- net at U23.16 (CH7): now also J7.1 (Pin_1); no longer J7.1 (Pin_1)
- net at U23.2 (CH9): now also J7.1 (Pin_1); no longer J7.1 (Pin_1)
- net at U23.3 (CH10): now also J7.1 (Pin_1)
- net at U23.4 (CH11): now also J7.1 (Pin_1); no longer J7.1 (Pin_1)
- net at U23.9 (CH0): now also J7.1 (Pin_1); no longer J7.1 (Pin_1)
- net at U20.4 (Y): now also JP1.1 (A); no longer D267.2 (DIN)
- new net: D267.2 (DIN), JP1.2 (C)
Other:
- moved on the sheet: J7
